File: Robotics Booster Pack.brd (EAGLE design)
At the start: 71.1 x 67.3 mm, 111 parts, among them U1 TPS62177.DQC, U11 SCHA4B0400, U13 XBEE-1B3, U14 TPS5450, U2 PCA9538.RGV, U3 DRV8800, U4 DRV8800, U5 DRV8800, U6 DRV8800, U8 MPU-6050, U9 INA220.DGS

Commit message: Exported BoM. Moved around schematic and renamed parts to be contiguous
Parts:
- removed C31, C33: .1uF, standardparts:0603
- removed C32: 2.2uF, standardparts:0603
- removed C41: 10nF, standardparts:0603
- removed C42: 10uF, standardparts:1206
- removed R17: 10k, standardparts:0603
- removed R18: 3.24k, standardparts:0603
- removed U14: TPS5450, packages(ti):DDA
- added C12, C16, C18, C20, C9: .1uF, standardparts:0603
- added R8: 2.2k, standardparts:0603
- added R9: 1k, standardparts:0603
- added U7: DRV8800, packages(ti):RTY.16
- C1: value (none) -> 220uF
- C10, C11: value (none) -> .1uF; device adafruit:PANASONIC_E -> standardparts:0603
- C13, C14: value 1uF -> .1uF
- C15: value 1uF -> 100uF; device standardparts:0603 -> adafruit:PANASONIC_E
- C23: value .1uF -> 2.2uF
- C26, C28, C30: value .1uF -> 1uF
- C3: value (none) -> 22uF; device adafruit:PANASONIC_E -> standardparts:0805
- C4: value 22uF -> 220uF; device standardparts:0805 -> adafruit:PANASONIC_E
- C5: value .1uF -> 10uF; device standardparts:0603 -> standardparts:1206
- C6: value .1uF -> 10nF
- C7: value .1uF -> 330uF; device standardparts:0603 -> adafruit:PANASONIC_E
- C8: value (none) -> 100uF
- Q1: value (none) -> FDMA3028N
- R3: value 1.5k -> 10k
- R4: value 1k -> 3.24k
- R5: value 10k -> 1.5k
- R6: value 2.2k -> 10k
- U1: value TPS62177.DQC -> INA220.DGS; device packages(ti):DQC -> packages(ti):DGS.10
- U2: value PCA9538.RGV -> TPS62177.DQC; device packages(ti):RGV.16 -> packages(ti):DQC
- U3: value DRV8800 -> TPS5450; device packages(ti):RTY.16 -> packages(ti):DDA
- U8: value MPU-6050 -> PCA9538.RGV; device invensense:QFN.24.4X4 -> packages(ti):RGV.16
- U9: value INA220.DGS -> MPU-6050; device packages(ti):DGS.10 -> invensense:QFN.24.4X4
- moved C25 50.8 mm to (40.3, 0.95), turned to 180 degrees
- moved C13 49.6 mm to (27.6, 50.2), turned to 270 degrees
- moved R5 48.3 mm to (5.71, 42.5), turned to 0 degrees
- moved C26 48.2 mm to (40.3, 2.22), turned to 180 degrees
- moved C15 47.4 mm to (54.6, 61.6), turned to 270 degrees
- moved R6 41.0 mm to (53.3, 50.5)
- moved U1 39.1 mm to (54.6, 54.6), turned to 270 degrees
- moved U9 38.7 mm to (35.6, 21.0), turned to 90 degrees
- moved C8 36.2 mm to (16.5, 61.6), turned to 270 degrees
- moved C24 34.5 mm to (39.4, 21.6), turned to 90 degrees
- moved C14 33.5 mm to (22.5, 55.6)
- moved C23 32.3 mm to (32.1, 22.2)
- moved U8 31.0 mm to (14.0, 43.2), turned to 180 degrees
- moved R4 30.9 mm to (34.3, 28.9)
- moved C5 30.2 mm to (40.0, 31.1), turned to 270 degrees
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- renumbered D6 to D2, H30 to H24, H31 to H27, L3 to L2, U13 to U10
Connections:
- net !RST: now also U8.1; no longer U2.1
- net 3.3V: now also C25.1, C26.1, C27.1, C28.1, C29.1, C3.1, C30.1, C4.+, R8.1, U1.6, U2.10, U2.8, U8.14, U9.13, U9.8; no longer C13.1, C14.1, C15.1, C3.+, C4.1, C5.1, C6.1, C7.1, R5.1, U1.10, U1.8, U2.14, U8.13, U8.8, U9.6
- net 5.0V: now also C7.+, R3.2; no longer C8.+, R17.2
- net FET0.G: now also U8.9; no longer U2.9
- net FET1.G: now also U8.10; no longer U2.10
- net GND: now also C10.1, C11.2, C13.1, C15.-, C17.1, C18.2, C20.1, C21.2, C23.2, C25.2, C26.2, C27.2, C3.2, C4.-, C7.-, R4.1, R5.2, U1.2, U1.7, U2.1, U2.5, U3.6, U7.12, U7.2, U7.7, U7.PAD, U8.15, U8.16, U8.6, U8.PAD, U9.11, U9.18, U9.9; no longer C10.-, C11.-, C13.2, C15.2, C25.1, C26.1, C27.1, C3.-, C31.2, C32.2, C33.1, C4.2, C42.2, C6.2, C7.2, R18.1, R3.2, U1.5, U1.6, U1.PAD, U14.6, U14.PAD, U2.15, U2.16, U3.12, U3.2, U3.7, U8.1, U8.11, U8.18, U8.9, U9.2, U9.7
- net IMU.INT: now also U8.8, U9.12; no longer U2.8, U8.12
- net M.MODE: now also R6.2, U7.16; no longer R5.2, U3.16
- net M0+: now also U4.9; no longer U5.9
- net M0-: now also U4.6; no longer U5.6
- net M0.EN: now also U4.3, U8.5; no longer U2.5, U5.3
- net M1+: now also U5.9; no longer U6.9
- net M1-: now also U5.6; no longer U6.6
- net M1.EN: now also U5.3, U8.4; no longer U2.4, U6.3
- net M2+: now also U6.9; no longer U3.9
- net M2-: now also U6.6; no longer U3.6
- net M2.EN: now also U6.3, U8.3; no longer U2.3, U3.3
- net M3+: now also U7.9; no longer U4.9
- net M3-: now also U7.6; no longer U4.6
- net M3.EN: now also U7.3, U8.2; no longer U2.2, U4.3
- net N$1: now also U2.9; no longer U1.9
- net N$13: now also C9.1, U4.11; no longer C17.1, U5.11
- net N$18: now also C10.2, U4.13; no longer C24.2, U5.13
- net N$19: now also C13.2, U5.13; no longer C25.2, U6.13
- net N$20: now also C17.2, U6.13; no longer C26.2, U3.13
- net N$21: now also C20.2, U7.13; no longer C27.2, U4.13
- net N$22: now also U1.10; no longer U9.10
- net N$24: now also C23.1, U9.20; no longer C32.1, U8.20
- net N$25: now also C12.1, U5.11; no longer C19.1, U6.11
- net N$27: now also C16.1, U6.11; no longer C21.1, U3.11
- net N$29: now also C19.1, U7.11; no longer C23.1, U4.11
- net N$3: now also R5.1; no longer R3.1
- net N$33: now also C6.1, U3.1; no longer C41.1, U14.1
- net N$34: now also C6.2, U3.8; no longer C41.2, U14.8
- net N$35: now also R3.1, R4.2, U3.4; no longer R17.1, R18.2, U14.4
- net N$37: now also C16.2, U6.10; no longer C21.2, U3.10
- net N$38: now also C9.2, U4.10; no longer C17.2, U5.10
- net N$39: now also C12.2, U5.10; no longer C19.2, U6.10
- net N$4: now also R9.2; no longer R4.2
- net N$40: now also C19.2, U7.10; no longer C23.2, U4.10
- net N$7: now also C24.2, U9.10; no longer C33.2, U8.10
- net N$8: now also U8.11; no longer U2.11
- net PA6: now also U5.4; no longer U6.4
- net PA7: now also U4.4; no longer U5.4
- net PB2: now also R8.2, U1.5, U8.12, U9.23; no longer R6.2, U2.12, U8.23, U9.5
- net PB3: now also U1.4, U8.13, U9.24; no longer U2.13, U8.24, U9.4
- net PC4: now also U4.1; no longer U5.1
- net PC7: now also U6.1; no longer U3.1
- net PD0: now also U7.4; no longer U4.4
- net PD1: now also U6.4; no longer U3.4
- net PF0: now also U5.1; no longer U6.1
- net PF3: now also U7.1; no longer U4.1
- net VBAT: now also C5.1, U1.8, U1.9, U2.2, U2.3, U3.7; no longer C42.1, U1.2, U1.3, U14.7, U9.8, U9.9
- net VMOTOR: now also C11.1, C14.1, C15.+, C18.1, C21.1, C8.+, U7.8; no longer C10.+, C11.+, C28.1, C29.1, C30.1, C31.1, U3.8
- net XBEE.CONNECTED: now also R9.1, U8.7; no longer R4.1, U2.7
