File: Robotics Booster Pack.sch (EAGLE design)
At the start: 111 parts, among them U1 TPS62177.DQC, U11 SCHA4B0400, U13 XBEE-1B3, U14 TPS5450, U2 PCA9538.RGV, U3 DRV8800, U4 DRV8800, U5 DRV8800, U6 DRV8800, U8 MPU-6050, U9 INA220.DGS

Commit message: Exported BoM. Moved around schematic and renamed parts to be contiguous
Parts:
- removed C31, C33: .1uF, standardparts:CAPACITOR.0603
- removed C32: 2.2uF, standardparts:CAPACITOR.0603
- removed C41: 10nF, standardparts:CAPACITOR.0603
- removed C42: 10uF, standardparts:CAPACITOR.1206
- removed D6: CDBC5XXX-G, comchip:CDBC5XXX-G
- removed H31: 1X3.4DB, te-connectivity:1X3.4DB
- removed L3: 10uH, coilcraft:INDUCTOR.XAL6060
- removed R17: 10k, standardparts:RESISTOR.0603
- removed R18: 3.24k, standardparts:RESISTOR.0603
- removed U13: XBEE-1B3, SparkFun-RF:XBEE-1B3
- removed U14: TPS5450, packages(ti):TPS54X0
- added C12, C16, C18, C20, C9: .1uF, standardparts:CAPACITOR.0603
- added D2: CDBC5XXX-G, comchip:CDBC5XXX-G
- added H27: 1X3.4DB, te-connectivity:1X3.4DB
- added L2: 10uH, coilcraft:INDUCTOR.XAL6060
- added R8: 2.2k, standardparts:RESISTOR.0603
- added R9: 1k, standardparts:RESISTOR.0603
- added U10: XBEE-1B3, SparkFun-RF:XBEE-1B3
- added U7: DRV8800, packages(ti):DRV8800.RTY
- C1: value (none) -> 220uF
- C10, C11: value (none) -> .1uF; device adafruit:CPOL-USE -> standardparts:CAPACITOR.0603
- C13, C14: value 1uF -> .1uF
- C15: value 1uF -> 100uF; device standardparts:CAPACITOR.0603 -> adafruit:CPOL-USE
- C23: value .1uF -> 2.2uF
- C26, C28, C30: value .1uF -> 1uF
- C3: value (none) -> 22uF; device adafruit:CPOL-USE -> standardparts:CAPACITOR.0805
- C4: value 22uF -> 220uF; device standardparts:CAPACITOR.0805 -> adafruit:CPOL-USE
- C5: value .1uF -> 10uF; device standardparts:CAPACITOR.0603 -> standardparts:CAPACITOR.1206
- C6: value .1uF -> 10nF
- C7: value .1uF -> 330uF; device standardparts:CAPACITOR.0603 -> adafruit:CPOL-USE
- C8: value (none) -> 100uF
- Q1: value (none) -> FDMA3028N
- R3: value 1.5k -> 10k
- R4: value 1k -> 3.24k
- R5: value 10k -> 1.5k
- R6: value 2.2k -> 10k
- U1: value TPS62177.DQC -> INA220.DGS; device packages(ti):TPS62177.DQC -> packages(ti):INA220.DGS
- U2: value PCA9538.RGV -> TPS62177.DQC; device packages(ti):PCA9538.RGV -> packages(ti):TPS62177.DQC
- U3: value DRV8800 -> TPS5450; device packages(ti):DRV8800.RTY -> packages(ti):TPS54X0
- U8: value MPU-6050 -> PCA9538.RGV; device invensense:MPU-6050 -> packages(ti):PCA9538.RGV
- U9: value INA220.DGS -> MPU-6050; device packages(ti):INA220.DGS -> invensense:MPU-6050
- renumbered H30 to H24
Connections:
- net !RST: now also U8.!RST; no longer U2.!RST
- net 3.3V: now also C25.1, C26.1, C27.1, C28.1, C29.1, C3.1, C30.1, C4.+, R8.1, U1.VS, U10.VDD, U2.SLEEP, U2.VOS, U8.VCC, U9.VDD, U9.VLOGIC; no longer C13.1, C14.1, C15.1, C3.+, C4.1, C5.1, C6.1, C7.1, R5.1, U1.SLEEP, U1.VOS, U13.VDD, U2.VCC, U8.VDD, U8.VLOGIC, U9.VS
- net 5.0V: now also C7.+, L2.2, R3.2; no longer C8.+, L3.2, R17.2
- net FET0.G: now also U8.P6; no longer U2.P6
- net FET1.G: now also U8.P7; no longer U2.P7
- net GND: now also C10.1, C11.2, C13.1, C15.-, C17.1, C18.2, C20.1, C21.2, C23.2, C25.2, C26.2, C27.2, C3.2, C4.-, C7.-, D2.2, H27.3, R4.1, R5.2, U1.A0, U1.A1, U1.GND, U10.GND, U2.AGND, U2.FB, U2.PGND, U7.GND, U7.SENSE, U8.A0, U8.A1, U9.AD0, U9.CLKIN, U9.FSYNC; no longer C10.-, C11.-, C13.2, C15.2, C25.1, C26.1, C27.1, C3.-, C31.2, C32.2, C33.1, C4.2, C42.2, C6.2, C7.2, D6.2, H31.3, R18.1, R3.2, U1.AGND, U1.FB, U1.PGND, U13.GND, U14.GND, U2.A0, U2.A1, U2.GND, U3.SENSE, U8.AD0, U8.CLKIN, U8.FSYNC, U9.A0, U9.A1
- net IMU.INT: now also U8.P5, U9.INT; no longer U2.P5, U8.INT
- net M.MODE: now also R6.2, U7.MODE; no longer R5.2, U3.MODE
- net M0+: now also U4.OUT-; no longer U5.OUT-
- net M0-: now also U4.OUT+; no longer U5.OUT+
- net M0.EN: now also U4.!SLEEP, U8.P3; no longer U2.P3, U5.!SLEEP
- net M1+: now also U5.OUT-; no longer U6.OUT-
- net M1-: now also U5.OUT+; no longer U6.OUT+
- net M1.EN: now also U5.!SLEEP, U8.P2; no longer U2.P2, U6.!SLEEP
- net M2+: now also U6.OUT-; no longer U3.OUT-
- net M2-: now also U6.OUT+; no longer U3.OUT+
- net M2.EN: now also U6.!SLEEP, U8.P1; no longer U2.P1, U3.!SLEEP
- net M3+: now also U7.OUT-; no longer U4.OUT-
- net M3-: now also U7.OUT+; no longer U4.OUT+
- net M3.EN: now also U7.!SLEEP, U8.P0; no longer U2.P0, U4.!SLEEP
- net N$1: now also U2.SW; no longer U1.SW
- net N$13: now also C9.1, U4.CP2; no longer C17.1, U5.CP2
- net N$18: now also C10.2, U4.VCP; no longer C24.2, U5.VCP
- net N$19: now also C13.2, U5.VCP; no longer C25.2, U6.VCP
- net N$20: now also C17.2, U6.VCP; no longer C26.2, U3.VCP
- net N$21: now also C20.2, U7.VCP; no longer C27.2, U4.VCP
- net N$22: now also H27.2, U1.VIN+; no longer H31.2, U9.VIN+
- net N$24: now also C23.1, U9.CPOUT; no longer C32.1, U8.CPOUT
- net N$25: now also C12.1, U5.CP2; no longer C19.1, U6.CP2
- net N$27: now also C16.1, U6.CP2; no longer C21.1, U3.CP2
- net N$29: now also C19.1, U7.CP2; no longer C23.1, U4.CP2
- net N$3: now also R5.1; no longer R3.1
- net N$33: now also C6.1, U3.BOOT; no longer C41.1, U14.BOOT
- net N$34: now also C6.2, D2.1, L2.1, U3.PH; no longer C41.2, D6.1, L3.1, U14.PH
- net N$35: now also R3.1, R4.2, U3.VSENSE; no longer R17.1, R18.2, U14.VSENSE
- net N$37: now also C16.2, U6.CP1; no longer C21.2, U3.CP1
- net N$38: now also C9.2, U4.CP1; no longer C17.2, U5.CP1
- net N$39: now also C12.2, U5.CP1; no longer C19.2, U6.CP1
- net N$4: now also R9.2; no longer R4.2
- net N$40: now also C19.2, U7.CP1; no longer C23.2, U4.CP1
- net N$7: now also C24.2, U9.REGOUT; no longer C33.2, U8.REGOUT
- net N$8: now also U8.!INT; no longer U2.!INT
- net PA6: now also U5.ENABLE; no longer U6.ENABLE
- net PA7: now also U4.ENABLE; no longer U5.ENABLE
- net PB0: now also U10.DOUT; no longer U13.DOUT
- net PB1: now also U10.DIN; no longer U13.DIN
- net PB2: now also R8.2, U1.SCL; no longer R6.2, U2.SCL
- net PB3: now also U1.SDA; no longer U2.SDA
- net PC4: now also U4.PHASE; no longer U5.PHASE
- net PC7: now also U6.PHASE; no longer U3.PHASE
- net PD0: now also U7.ENABLE; no longer U4.ENABLE
- net PD1: now also U6.ENABLE; no longer U3.ENABLE
- net PF0: now also U5.PHASE; no longer U6.PHASE
- net PF3: now also U7.PHASE; no longer U4.PHASE
- net VBAT: now also C5.1, H27.1, U1.VBUS, U1.VIN-, U2.EN, U2.VIN, U3.VIN; no longer C42.1, H31.1, U1.EN, U1.VIN, U14.VIN, U9.VBUS, U9.VIN-
- net VMOTOR: now also C11.1, C14.1, C15.+, C18.1, C21.1, C8.+, U7.VMOT; no longer C10.+, C11.+, C28.1, C29.1, C30.1, C31.1, U3.VMOT
- net XBEE.CONNECTED: now also R9.1, U10.DIO9, U8.P4; no longer R4.1, U13.DIO9, U2.P4
Other:
- moved on the sheet: C1, C13, C14, C17, C19, C2, C21, C22, C23, C24, C25, C26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
